File: ftuno.kicad_sch (KiCad schematic)
At the start: 53 parts, among them CN1 AFC10-S04QCA-00, J1 USB_C_Receptacle_USB2.0_16P, J10 Conn_01x10_Socket, J11 Conn_01x08_Pin, J12 Conn_01x08_Socket, J13 DC050-T, J2 Conn_02x03_Odd_Even, J3 Conn_01x08_Pin, J4 Conn_01x08_Socket, J5 Conn_02x04_Odd_Even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

Commit message: use seperate resistors for led, use higher rns for level shifters
Parts:
- removed RN3: 2.2k, Resistor_SMD:R_Array_Convex_4x0603, symbol Device:R_Pack04_Split
- added R11, R12, R6, R7: 2.2k, Resistor_SMD:R_0402_1005Metric, symbol Device:R
- RN1, RN2: value 2.2k -> 4.7k
Connections:
- net GND: now also R12.2, R6.2
- net RX0: now also R7.2
- net TX1: now also R11.2
- net at LED3.1 (K): now also R11.1
- net at LED4.1 (K): now also R12.1
- net at LED2.1 (K): now also R7.1
- net at LED1.1 (K): now also R6.1
